Commit message: set model materials, add velodyne hdl-16 lidar

File: src/amiga_description/urdf/amiga.urdf (robot description, URDF)
Before this commit: robot robot_with_wheels, 22 links, 21 joints
Links:
- removed link amiga_chase
- added link base_link
- added link chassis_link
- added link imu_link, mass 0.001
- added link navsat_link; visual cylinder length=0.016 radius=0.026
- added link velodyne, mass 0.01; collision sphere radius=0; visual mesh filename=package://velodyne_description/meshes/VLP16_scan.dae
- link smartfork1: mass 0.1 -> 40
- link smartfork2: mass 0.1 -> 40
- link smartfork3: mass 0.1 -> 40
- link smartfork4: mass 0.1 -> 40
- link wheel1: mass 0.1 -> 15
- link wheel2: mass 0.1 -> 15
- link wheel3: mass 0.1 -> 15
- link wheel4: mass 0.1 -> 15
Joints:
- added joint base_link_joint: type fixed, parent base_link, child chassis_link, origin xyz=0 0 0 rpy=0 0 0
- added joint imu_joint: type fixed, parent front_center, child imu_link
- added joint navsat_joint: type fixed, parent front_center, child navsat_link, origin xyz=0 0.2 0.036
- added joint velodyne_joint: type fixed, parent front_center, child velodyne, origin xyz=0 0 0.25 rpy=0 0 0
- joint wheel_0_joint: axis 0 0 1 -> 0 0 -1
- joint wheel_1_joint: axis 0 0 1 -> 0 0 -1
- joint wheel_2_joint: axis 0 0 1 -> 0 0 -1
- joint wheel_3_joint: axis 0 0 1 -> 0 0 -1
- joint world_joint: parent amiga_chase -> chassis_link

Commit message: modify the Amiga mass, add sensors (plugins) and two realsense

File: src/amiga_description/urdf/amiga.urdf (robot description, URDF)
Before this commit: robot robot_with_wheels, 26 links, 25 joints
Links:
- link smartfork1: mass 40 -> 15
- link smartfork2: mass 40 -> 15
- link smartfork3: mass 40 -> 15
- link smartfork4: mass 40 -> 15

Commit message: shrink the wdith, adjust parameters

File: src/amiga_description/urdf/amiga.urdf (robot description, URDF)
Before this commit: robot robot_with_wheels, 26 links, 25 joints
Links:
- link rig_12_left: mass 0.1 -> None
- link rig_12_right: mass 0.1 -> None
- link rig_13: mass 0.1 -> None; geometry collision box size=0.04 0.02 1.0; visual box size=0.04 0.02 1.0
- link rig_24: mass 0.1 -> None; geometry collision box size=0.04 0.02 1.0; visual box size=0.04 0.02 1.0
- link rig_34_left: mass 0.1 -> None
- link rig_34_right: mass 0.1 -> None
- link smartfork1: mass 15 -> ${smartfork_weight}
- link smartfork2: mass 15 -> ${smartfork_weight}
- link smartfork3: mass 15 -> ${smartfork_weight}
- link smartfork4: mass 15 -> ${smartfork_weight}
- link wheel1: mass 15 -> ${wheel_weight}
- link wheel2: mass 15 -> ${wheel_weight}
- link wheel3: mass 15 -> ${wheel_weight}
- link wheel4: mass 15 -> ${wheel_weight}
Joints:
- removed joint front_center_joint
- removed joint world_joint_fork1
- added joint front_center_to_smartfork1_joint: type fixed, parent front_center, child smartfork1, origin xyz=0 0.5 0 rpy=1.5708 0 0
- added joint front_center_to_smartfork3_joint: type fixed, parent front_center, child smartfork3, origin xyz=0 -0.5 0 rpy=1.5708 0 0
- joint base_link_joint: origin xyz=0 0 0 rpy=0 0 0 -> xyz=0.5 0 0 rpy=0 0 0
- joint imu_joint: parent front_center -> base_link
- joint rig_13_joint: origin xyz=0 0 -1.0 rpy=0 0 0 -> xyz=0 0 -0.5 rpy=0 0 0
- joint rig_24_joint: origin xyz=0 0 -1.0 rpy=0 0 0 -> xyz=0 0 -0.5 rpy=0 0 0

Commit message: shrink the amiga size

File: src/amiga_description/urdf/amiga.urdf (robot description, URDF)
Before this commit: robot robot_with_wheels, 26 links, 25 joints
Links:
- link front_laser: mass 1.1 -> None
- link imu_link: mass 0.001 -> None
- link rig_13: mass None -> 30
- link rig_24: mass None -> 30
- link velodyne: mass 0.01 -> None

Commit message: [Solved][ISSUE01] Change mesh package name from gazebo_ros to package://amiga_description/meshes

File: src/amiga_description/urdf/amiga.urdf (robot description, URDF)
Before this commit: robot robot_with_wheels, 26 links, 25 joints
Links:
- link link1_connector: geometry collision mesh filename=package://amiga_description/meshes/connector.stl; visual mesh filename=package://amiga_description/meshes/connector.stl
- link link2_connector: geometry collision mesh filename=package://amiga_description/meshes/connector.stl; visual mesh filename=package://amiga_description/meshes/connector.stl
- link link3_connector: geometry collision mesh filename=package://amiga_description/meshes/connector.stl; visual mesh filename=package://amiga_description/meshes/connector.stl
- link link4_connector: geometry collision mesh filename=package://amiga_description/meshes/connector.stl; visual mesh filename=package://amiga_description/meshes/connector.stl
- link smartfork1: geometry collision mesh filename=package://amiga_description/meshes/smartfork.stl scale=0.001 0.001 0.001; visual mesh filename=package://amiga_description/meshes/smartfork.stl scale=0.001 0.001 0.001
- link smartfork2: geometry collision mesh filename=package://amiga_description/meshes/smartfork.stl scale=0.001 0.001 0.001; visual mesh filename=package://amiga_description/meshes/smartfork.stl scale=0.001 0.001 0.001
- link smartfork3: geometry collision mesh filename=package://amiga_description/meshes/smartfork.stl scale=0.001 0.001 0.001; visual mesh filename=package://amiga_description/meshes/smartfork.stl scale=0.001 0.001 0.001
- link smartfork4: geometry collision mesh filename=package://amiga_description/meshes/smartfork.stl scale=0.001 0.001 0.001; visual mesh filename=package://amiga_description/meshes/smartfork.stl scale=0.001 0.001 0.001
- link wheel1: geometry collision mesh filename=package://amiga_description/meshes/smartfork_tire.stl scale=0.001 0.001 0.001; visual mesh filename=package://amiga_description/meshes/smartfork_tire.stl scale=0.001 0.001 0.001
- link wheel2: geometry collision mesh filename=package://amiga_description/meshes/smartfork_tire.stl scale=0.001 0.001 0.001; visual mesh filename=package://amiga_description/meshes/smartfork_tire.stl scale=0.001 0.001 0.001
- link wheel3: geometry collision mesh filename=package://amiga_description/meshes/smartfork_tire.stl scale=0.001 0.001 0.001; visual mesh filename=package://amiga_description/meshes/smartfork_tire.stl scale=0.001 0.001 0.001
- link wheel4: geometry collision mesh filename=package://amiga_description/meshes/smartfork_tire.stl scale=0.001 0.001 0.001; visual mesh filename=package://amiga_description/meshes/smartfork_tire.stl scale=0.001 0.001 0.001

Commit message: try to use rtabmap

File: src/amiga_description/urdf/amiga.urdf (robot description, URDF)
Before this commit: robot robot_with_wheels, 26 links, 25 joints
Links:
- link velodyne: geometry collision mesh filename=package://velodyne_description/meshes/VLP16_scan.dae; visual mesh filename=package://velodyne_description/meshes/VLP16_scan.dae

Commit message: regular update

File: src/amiga_description/urdf/amiga.urdf (robot description, URDF)
Before this commit: robot robot_with_wheels, 26 links, 25 joints
Links:
- removed link wheel4
- added link wheel0, mass ${wheel_weight}; collision cylinder length=${wheel_width} radius=${wheel_radius}; visual mesh filename=package://amiga_description/meshes/smartfork_tire.stl scale=0.001 0.001 0.001
- link front_laser: mass None -> 0.001
- link imu_link: mass None -> 0.001
- link rig_12_left: mass None -> 3.888
- link rig_12_right: mass None -> 3.888
- link rig_34_left: mass None -> 3.888
- link rig_34_right: mass None -> 3.888
- link velodyne: mass None -> 0.01
- link wheel1: geometry collision cylinder length=${wheel_width} radius=${wheel_radius}; visual mesh filename=package://amiga_description/meshes/smartfork_tire.stl scale=0.001 0.001 0.001
- link wheel2: geometry collision cylinder length=${wheel_width} radius=${wheel_radius}; visual mesh filename=package://amiga_description/meshes/smartfork_tire.stl scale=0.001 0.001 0.001
- link wheel3: geometry collision cylinder length=${wheel_width} radius=${wheel_radius}; visual mesh filename=package://amiga_description/meshes/smartfork_tire.stl scale=0.001 0.001 0.001
Joints:
- joint wheel_0_joint: child wheel1 -> wheel0
- joint wheel_1_joint: child wheel2 -> wheel1
- joint wheel_2_joint: child wheel3 -> wheel2
- joint wheel_3_joint: child wheel4 -> wheel3
