Commit message: optimize amiga model to xacro type and integrate model into one file

File: src/amiga_description/xacro/amiga.xacro (robot description, xacro)
@@ -1,695 +1,142 @@
 <?xml version="1.0" ?>
-<!-- =================================================================================== -->
-<!-- |    This document was autogenerated by xacro from urdf/amiga.urdf                | -->
-<!-- |    EDITING THIS FILE BY HAND IS NOT RECOMMENDED                                 | -->
-<!-- =================================================================================== -->
-<robot name="robot_with_wheels">
-  <material name="dark_grey">
-    <color rgba="  0.2 0.2 0.2 1.0"/>
-  </material>
-  <material name="light_grey">
-    <color rgba="0.4 0.4 0.4 1.0"/>
-  </material>
-  <material name="yellow">
-    <color rgba="0.8 0.8 0.0 1.0"/>
-  </material>
-  <material name="black">
-    <color rgba="0.15 0.15 0.15 1.0"/>
-  </material>
-  <link name="amiga_frame"/>
-  <!-- Define origin for the front_center frame -->
-  <joint name="world_joint" type="fixed">
-    <origin rpy="0 0 0" xyz="0 0.0 0.65"/>
-    <parent link="amiga_frame"/>
-    <child link="front_center"/>
-  </joint>
-  <link name="front_center"/>
-  <!-- Define origin for the front_center frame -->
-  <joint name="front_center_joint" type="fixed">
-    <origin rpy="1.5708 0 0" xyz="0 -1.0 0"/>
-    <parent link="front_center"/>
-    <child link="smartfork3"/>
-  </joint>
-  <link name="wheel3">
-    <visual>
-      <origin rpy="0 0 0" xyz="0 0.395 0"/>
-      <geometry>
-        <mesh filename="package://amiga_ros/amiga_description/smartfork_tire.stl" scale="0.001 0.001 0.001"/>
-      </geometry>
-    </visual>
-    <collision>
-      <origin rpy="0 0 0" xyz="0 0.395 0"/>
-      <geometry>
-        <mesh filename="package://amiga_ros/amiga_description/smartfork_tire.stl" scale="0.001 0.001 0.001"/>
-      </geometry>
-    </collision>
-    <inertial>
-      <mass value="0.1"/>
-      <origin rpy="0 0 0" xyz="0 0 0"/>
-      <inertia ixx="0.03" ixy="0.0" ixz="0.0" iyy="0.03" iyz="0.0" izz="0.03"/>
-    </inertial>
-  </link>
-  <gazebo reference="wheel3">
-    <material>Gazebo/DarkGrey</material>
-    <selfCollide>false</selfCollide>
-    <mu1 value="0.5"/>
-    <mu2 value="0.5"/>
-    <kp value="10000000.0"/>
-    <kd value="1"/>
-    <fdir1 value="1 0 0"/>
-    <plugin name="gazebo_ros_control">
-      <robotNamespace>/</robotNamespace>
-    </plugin>
-  </gazebo>
-  <link name="smartfork3">
-    <visual>
-      <geometry>
-        <mesh filename="package://amiga_ros/amiga_description/smartfork.stl" scale="0.001 0.001 0.001"/>
-      </geometry>
-    </visual>
-    <collision>
-      <geometry>
-        <mesh filename="package://amiga_ros/amiga_description/smartfork.stl" scale="0.001 0.001 0.001"/>
-      </geometry>
-    </collision>
-    <inertial>
-      <mass value="0.1"/>
-      <origin rpy="0 0 0" xyz="0 0 0"/>
-      <inertia ixx="0.03" ixy="0.0" ixz="0.0" iyy="0.03" iyz="0.0" izz="0.03"/>
-    </inertial>
-  </link>
-  <joint name="wheel_2_joint" type="continuous">
-    <parent link="smartfork3"/>
-    <child link="wheel3"/>
-    <origin rpy="0 0 0" xyz="0 -0.395 0"/>
-    <axis xyz="0 0 1"/>
-  </joint>
-  <!-- <transmission name="front_right_wheel_trans">
-        <type>transmission_interface/SimpleTransmission</type>
-        <joint name="wheel_2_joint">
-            <hardwareInterface>transmission_interface/VelocityJointInterface</hardwareInterface>
+<robot name="differential_drive_robot" xmlns:xacro="http://ros.org/wiki/xacro">
+    <material name="dark_grey">
+        <color rgba="0.2 0.2 0.2 1.0"/>
+    </material>
+    <material name="light_grey">
+        <color rgba="0.4 0.4 0.4 1.0"/>
+    </material>
+    <material name="yellow">
+        <color rgba="0.8 0.8 0.0 1.0"/>
+    </material>
+    <material name="black">
+        <color rgba="0.15 0.15 0.15 1.0"/>
+    </material>
+    <material name="aluminum">
+        <color rgba="0.8 0.85 0.88 1"/>
+    </material>
+    <material name="white">
+        <color rgba="1.0 1.0 1.0 1.0"/>
+    </material>
+    <xacro:property name="wheel_link_length" value="0.2" />
+    <xacro:property name="wheel_link_radius" value="0.215" />
+    <!-- Body Dimensions -->
+    <xacro:property name="body_link_x_dim" value="1.0"/>
+    <xacro:property name="body_link_y_dim" value="1.0"/>
+    <xacro:property name="body_link_z_dim" value="0.5"/>
+    <xacro:property name="wheel_link_z_location" value="0"/>
+    <xacro:property name="body_mass" value="300"/>
+    <xacro:property name="pi_constant" value="3.1415926"/>
+    <xacro:property name="wheel_mass" value="10"/>
+    <!-- Moments -->
+    <xacro:property name="Iz_wheel" value="${0.5 * wheel_mass * wheel_link_radius * wheel_link_radius}"/>
+    <xacro:property name="Ixy_wheel" value="${(1.0)/(12.0)*wheel_mass * (3.0 * wheel_link_radius * wheel_link_radius + wheel_link_length * wheel_link_length)}"/>
+    <xacro:property name="wheel_weight" value="3.0" />
+    <xacro:property name="wheel_radius" value="0.215" />
+    <xacro:property name="wheel_width" value="0.14" />
+    <xacro:property name="mu1" value="0.1" />
+    <xacro:property name="mu2" value="0.1" />
+    <xacro:macro name="inertia_wheel">
+        <inertial>
+            <origin xyz = "0 0 0" rpy="0 0 0"/>
+            <mass value="${wheel_mass}"/>
+            <inertia ixx="${Ixy_wheel}"  iyy="${Ixy_wheel}"  izz="${Iz_wheel}" ixy="0.0" ixz="0.0" iyz="0.0"/>
+        </inertial>
+    </xacro:macro>
+    <xacro:include filename="$(find amiga_description)/urdf/amiga.new.gazebo"/>
+    <!-- define the base link -->
+    <link name="dummy"/>
+    <joint name="dummy_joint" type="fixed">
+        <parent link="dummy"/>
+        <child link="body_link"/>
+    </joint>
+    <link name="body_link">
+        <visual>
+            <origin xyz="0 0 0" rpy="0 0 0" />
+            <geometry>
+                <mesh filename="package://amiga_description/meshes/amiga_base.stl" scale="1 1 1" />
+                <!-- <mesh filename="package://amiga_description/meshes/amiga_base.stl" scale="0.001 0.001 0.001" /> -->
+            </geometry>
+        </visual>
+        <collision>
+            <origin xyz="0 0 0" rpy="0 0 0" />
+            <geometry>
+                <mesh filename="package://amiga_description/meshes/amiga_base.stl" scale="1 1 1" />
+                <!-- <mesh filename="package://amiga_description/meshes/amiga_base.stl" scale="0.001 0.001 0.001" /> -->
+            </geometry>
+        </collision>
+        <inertial>
+            <origin xyz="0 0 0.4" rpy="0 0 0" />
+            <mass value="335.0"/>
+            <inertia    ixx="94.59"
+                        iyy="94.03"
+                        izz="171.3"
+                        ixy="0.001581"
+                        ixz="-0.02401"
+                        iyz="0.003946"/>
+        </inertial>
+    </link>
+    <xacro:macro name="wheel" params="prefix *joint_pose">
+        <joint name="wheel${prefix}_joint" type="continuous">
+            <parent link="body_link"/>
+            <child link="wheel${prefix}_link"/>
+            <xacro:insert_block name="joint_pose"/>
+            <axis xyz="0 0 -1"/>
+            <limit effort="1000" velocity="1000"/>
+            <dynamic damping="1.0" friction="1.0"/>
         </joint>
-        <actuator name="front_right_actuator">
-            <mechanicalReduction>1</mechanicalReduction>
-            <hardwareInterface>transmission_interface/VelocityJointInterface</hardwareInterface>
-        </actuator>
-    </transmission> -->
-  <!-- <transmission name="front_right_wheel_trans" type="SimpleTransmission">
-      <actuator name="front_right_actuator"/>
-      <joint name="wheel_2_joint"/>
-      <mechanicalReduction>1</mechanicalReduction>
-      <motorTorqueConstant>1</motorTorqueConstant>
-    </transmission> -->
-  <link name="rig_34_left">
-    <visual>
-      <geometry>
-        <box size="1.2 0.04 0.03"/>
-      </geometry>
-      <origin rpy="1.5708 0.0 0.0" xyz="-0.5 0 0"/>
-    </visual>
-    <collision>
-      <geometry>
-        <box size="1.2 0.04 0.03"/>
-      </geometry>
-      <origin rpy="1.5708 0.0 0.0" xyz="-0.5 0 0"/>
-    </collision>
-    <inertial>
-      <mass value="0.1"/>
-      <origin rpy="0 0 0" xyz="0 0 0"/>
-      <inertia ixx="0.03" ixy="0.0" ixz="0.0" iyy="0.03" iyz="0.0" izz="0.03"/>
-    </inertial>
-  </link>
-  <link name="rig_34_right">
-    <visual>
-      <geometry>
-        <box size="1.2 0.04 0.03"/>
-      </geometry>
-      <origin rpy="1.5708 0.0 0.0" xyz="-0.5 0 0"/>
-    </visual>
-    <collision>
-      <geometry>
-        <box size="1.2 0.04 0.03"/>
-      </geometry>
-      <origin rpy="1.5708 0.0 0.0" xyz="-0.5 0 0"/>
-    </collision>
-    <inertial>
-      <mass value="0.1"/>
-      <origin rpy="0 0 0" xyz="0 0 0"/>
-      <inertia ixx="0.03" ixy="0.0" ixz="0.0" iyy="0.03" iyz="0.0" izz="0.03"/>
-    </inertial>
-  </link>
-  <joint name="rig34_right" type="fixed">
-    <parent link="smartfork3"/>
-    <child link="rig_34_left"/>
-    <origin rpy="-1.5708 0 0" xyz="0 -0.03 0.06"/>
-  </joint>
-  <joint name="rig34_left" type="fixed">
-    <parent link="smartfork3"/>
-    <child link="rig_34_right"/>
-    <origin rpy="-1.5708 0 0" xyz="0 -0.03 -0.06"/>
-  </joint>
-  <link name="wheel4">
-    <visual>
-      <origin rpy="0 0 0" xyz="0 0.395 0"/>
-      <geometry>
-        <mesh filename="package://amiga_ros/amiga_description/smartfork_tire.stl" scale="0.001 0.001 0.001"/>
-      </geometry>
-    </visual>
-    <collision>
-      <origin rpy="0 0 0" xyz="0 0.395 0"/>
-      <geometry>
-        <mesh filename="package://amiga_ros/amiga_description/smartfork_tire.stl" scale="0.001 0.001 0.001"/>
-      </geometry>
-    </collision>
-    <inertial>
-      <mass value="0.1"/>
-      <origin rpy="0 0 0" xyz="0 0 0"/>
-      <inertia ixx="0.03" ixy="0.0" ixz="0.0" iyy="0.03" iyz="0.0" izz="0.03"/>
-    </inertial>
-  </link>
-  <gazebo reference="wheel4">
-    <material>Gazebo/DarkGrey</material>
-    <selfCollide>false</selfCollide>
-    <mu1 value="0.5"/>
-    <mu2 value="0.5"/>
-    <kp value="10000000.0"/>
-    <kd value="1"/>
-    <fdir1 value="1 0 0"/>
-  </gazebo>
-  <link name="smartfork4">
-    <visual>
-      <geometry>
-        <mesh filename="package://amiga_ros/amiga_description/smartfork.stl" scale="0.001 0.001 0.001"/>
-      </geometry>
-    </visual>
-    <collision>
-      <geometry>
-        <mesh filename="package://amiga_ros/amiga_description/smartfork.stl" scale="0.001 0.001 0.001"/>
-      </geometry>
-    </collision>
-    <inertial>
-      <mass value="0.1"/>
-      <origin rpy="0 0 0" xyz="0 0 0"/>
-      <inertia ixx="0.03" ixy="0.0" ixz="0.0" iyy="0.03" iyz="0.0" izz="0.03"/>
-    </inertial>
-  </link>
-  <joint name="smartfork_34" type="fixed">
-    <origin rpy="0 0 0" xyz="-1.0 0 0"/>
-    <parent link="smartfork3"/>
-    <child link="smartfork4"/>
-  </joint>
-  <joint name="wheel_3_joint" type="continuous">
-    <parent link="smartfork4"/>
-    <child link="wheel4"/>
-    <origin rpy="0 0 0" xyz="0 -0.395 0"/>
-    <axis xyz="0 0 1"/>
-  </joint>
-  <!-- In reality, Jackal has only two motors, one per side. However, it's more
-         straightforward for Gazebo to simulate as if there's an actuator per wheel. -->
-  <!-- <transmission name="rear_right_wheel_trans">
-        <type>transmission_interface/SimpleTransmission</type>
-        <joint name="wheel_3_joint">
-            <hardwareInterface>transmission_interface/VelocityJointInterface</hardwareInterface>
-        </joint>
-        <actuator name="rear_right_actuator">
-            <mechanicalReduction>1</mechanicalReduction>
-            <hardwareInterface>transmission_interface/VelocityJointInterface</hardwareInterface>
-        </actuator>
-    </transmission> -->
-  <!--
-    <transmission name="rear_right_wheel_trans" type="SimpleTransmission">
-      <actuator name="rear_right_actuator"/>
-      <joint name="wheel_3_joint"/>
-      <mechanicalReduction>1</mechanicalReduction>
-      <motorTorqueConstant>1</motorTorqueConstant>
-    </transmission> -->
-  <link name="link3_connector">
-    <visual>
-      <geometry>
-        <mesh filename="package://amiga_ros/amiga_description/connector.stl"/>
-      </geometry>
-      <origin rpy="0 0 0" xyz="0 0 -0.01"/>
-    </visual>
-    <collision>
-      <geometry>
-        <mesh filename="package://amiga_ros/amiga_description/connector.stl"/>
-      </geometry>
-      <origin rpy="0 0 0" xyz="0 0 -0.01"/>
-    </collision>
-    <inertial>
-      <mass value="0.1"/>
-      <origin rpy="0 0 0" xyz="0 0 0"/>
-      <inertia ixx="0.03" ixy="0.0" ixz="0.0" iyy="0.03" iyz="0.0" izz="0.03"/>
-    </inertial>
-  </link>
-  <joint name="link3_connector_joint" type="fixed">
-    <parent link="smartfork3"/>
-    <child link="link3_connector"/>
-    <origin rpy="0 0 0" xyz="0 0 0"/>
-  </joint>
-  <link name="rig_13">
-    <visual>
-      <geometry>
-        <box size="0.04 0.02 2.0"/>
-      </geometry>
-      <origin rpy="0 0.0 0.0" xyz="0 0.02 0"/>
-    </visual>
-    <collision>
-      <geometry>
-        <box size="0.04 0.02 2.0"/>
-      </geometry>
-      <origin rpy="0 0.0 0.0" xyz="0 0.02 0"/>
-    </collision>
-    <inertial>
-      <mass value="0.1"/>
-      <origin rpy="0 0 0" xyz="0 0 0"/>
-      <inertia ixx="0.03" ixy="0.0" ixz="0.0" iyy="0.03" iyz="0.0" izz="0.03"/>
-    </inertial>
-  </link>
-  <joint name="rig_13_joint" type="fixed">
-    <parent link="link3_connector"/>
-    <child link="rig_13"/>
-    <origin rpy="0 0 0" xyz="0 0 -1.0"/>
-  </joint>
-  <link name="link4_connector">
-    <visual>
-      <geometry>
-        <mesh filename="package://amiga_ros/amiga_description/connector.stl"/>
-      </geometry>
-      <origin rpy="0 0 0" xyz="0 0 -0.01"/>
-    </visual>
-    <collision>
-      <geometry>
-        <mesh filename="package://amiga_ros/amiga_description/connector.stl"/>
-      </geometry>
-      <origin rpy="0 0 0" xyz="0 0 -0.01"/>
-    </collision>
-    <inertial>
-      <mass value="0.1"/>
-      <origin rpy="0 0 0" xyz="0 0 0"/>
-      <inertia ixx="0.03" ixy="0.0" ixz="0.0" iyy="0.03" iyz="0.0" izz="0.03"/>
-    </inertial>
-  </link>
-  <joint name="link4_connector_joint" type="fixed">
-    <parent link="smartfork4"/>
-    <child link="link4_connector"/>
-    <origin rpy="0 0 0" xyz="0 0 0"/>
-  </joint>
-  <link name="rig_24">
-    <visual>
-      <geometry>
-        <box size="0.04 0.02 2.0"/>
-      </geometry>
-      <origin rpy="0 0.0 0.0" xyz="0 0.02 0"/>
-    </visual>
-    <collision>
-      <geometry>
-        <box size="0.04 0.02 2.0"/>
-      </geometry>
-      <origin rpy="0 0.0 0.0" xyz="0 0.02 0"/>
-    </collision>
-    <inertial>
-      <mass value="0.1"/>
-      <origin rpy="0 0 0" xyz="0 0 0"/>
-      <inertia ixx="0.03" ixy="0.0" ixz="0.0" iyy="0.03" iyz="0.0" izz="0.03"/>
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
Commit message: Add transmission EffortJointInterface and gazebo_ros_control

File: src/amiga_description/xacro/amiga.xacro (robot description, xacro)
@@ -44,5 +44,5 @@
         </inertial>
     </xacro:macro>
-    <xacro:include filename="$(find amiga_description)/urdf/amiga.new.gazebo"/>
+    <xacro:include filename="$(find amiga_description)/urdf/amiga.gazebo"/>
     <!-- define the base link -->
     <link name="dummy"/>
@@ -101,4 +101,21 @@
             <xacro:inertia_wheel/>
         </link>
+        <gazebo reference = "wheel${prefix}_link">
+            <mu1>${mu1}</mu1>
+            <mu2>${mu1}</mu2>
+            <kp value="10000000.0" />
+            <kd value="1" />
+            <fdir1 value="1 0 0"/>
+            <material>Gazebo/Gray</material>
+        </gazebo>
+        <transmission name="${prefix}_wheel_trans">
+            <type>transmission_interface/SimpleTransmission</type>
+            <joint name="wheel${prefix}_joint">
+                <hardwareInterface>hardware_interface/EffortJointInterface</hardwareInterface>
+            </joint>
+            <actuator name="${prefix}_actuator">
+                <mechanicalReduction>1</mechanicalReduction>
+            </actuator>
+        </transmission>
     </xacro:macro>
     <xacro:wheel prefix="1">
@@ -138,5 +155,5 @@
         <parent link="body_link"/>
         <child link="navsat_link"/>
-        <origin xyz="0.5 0.0 1.0"/>
+        <origin xyz="0.5 0.0 0.6"/>
     </joint>
 </robot>

Commit message: corresponding modification with PID control function

File: src/amiga_description/xacro/amiga.xacro (robot description, xacro)
@@ -35,6 +35,6 @@
     <xacro:property name="wheel_radius" value="0.215" />
     <xacro:property name="wheel_width" value="0.14" />
-    <xacro:property name="mu1" value="0.1" />
-    <xacro:property name="mu2" value="0.1" />
+    <xacro:property name="mu1" value="1.0" />
+    <xacro:property name="mu2" value="1.0" />
     <xacro:macro name="inertia_wheel">
         <inertial>

Commit message: optimized mu1=1 mu2=0.3 torque=2500

File: src/amiga_description/xacro/amiga.xacro (robot description, xacro)
@@ -35,6 +35,6 @@
     <xacro:property name="wheel_radius" value="0.215" />
     <xacro:property name="wheel_width" value="0.14" />
-    <xacro:property name="mu1" value="1.0" />
-    <xacro:property name="mu2" value="1.0" />
+    <xacro:property name="mu1" value="1" />
+    <xacro:property name="mu2" value="0.3" />
     <xacro:macro name="inertia_wheel">
         <inertial>
@@ -77,5 +77,5 @@
         </inertial>
     </link>
-    <xacro:macro name="wheel" params="prefix *joint_pose">
+    <xacro:macro name="wheel" params="prefix *joint_pose    ">
         <joint name="wheel${prefix}_joint" type="continuous">
             <parent link="body_link"/>
@@ -103,10 +103,14 @@
         <gazebo reference = "wheel${prefix}_link">
             <mu1>${mu1}</mu1>
-            <mu2>${mu1}</mu2>
-            <kp value="10000000.0" />
+            <mu2>${mu2}</mu2>
+            <kp value="100000000.0" />
             <kd value="1" />
             <fdir1 value="1 0 0"/>
             <material>Gazebo/Gray</material>
         </gazebo>
+        <!-- <gazebo reference="wheel${prefix}_joint">
+            <stopKd value="1000000.0" />
+            <stopKp value="1000000.0" />
+        </gazebo> -->
         <transmission name="${prefix}_wheel_trans">
             <type>transmission_interface/SimpleTransmission</type>

Commit message: Add Depth camera and Velodyne (GPU) version

File: src/amiga_description/xacro/amiga.xacro (robot description, xacro)
@@ -35,6 +35,7 @@
     <xacro:property name="wheel_radius" value="0.215" />
     <xacro:property name="wheel_width" value="0.14" />
-    <xacro:property name="mu1" value="1" />
-    <xacro:property name="mu2" value="0.3" />
+    <xacro:property name="mu1" value="2" />
+    <xacro:property name="mu2" value="0.1" />
+    <xacro:property name="gpu_lidar" value="true"/>
     <xacro:macro name="inertia_wheel">
         <inertial>
@@ -159,5 +160,32 @@
         <parent link="body_link"/>
         <child link="navsat_link"/>
-        <origin xyz="0.5 0.0 0.6"/>
+        <origin xyz="0.5 0.1 0.65"/>
     </joint>
+    <link name="velodyne_holder_link">
+        <visual>
+            <geometry>
+                <cylinder length="0.2" radius="0.036"/>
+            </geometry>
+            <origin xyz="0 0 0.1"/>
+            <material name="black"/>
+        </visual>
+    </link>
+    <joint name="velodyne_holder_joint" type="fixed">
+        <parent link="body_link"/>
+        <child link="velodyne_holder_link"/>
+        <origin xyz="0.5 0.0 0.65"/>
+    </joint>
+    <!-- Add the Velodyne HDL-16 -->
+    <xacro:include filename="$(find velodyne_description)/urdf/VLP-16.urdf.xacro"/>
+    <xacro:VLP-16 parent="velodyne_holder_link" name="velodyne" topic="/velodyne_points" hz="10" samples="440" gpu="${gpu_lidar}">
+        <origin xyz="0.0 0.0 0.2" rpy="0 0 0" />
+    </xacro:VLP-16>
+    <!-- Add the Left Depth Camera -->
+  <xacro:include filename="$(find realsense2_description_gazebo)/urdf/_d435.urdf.xacro" />
+  <xacro:sensor_d435 name="camera_left" topics_ns="camera_left" parent="body_link" publish_pointcloud="true">
+    <origin xyz="0.5 -0.1 0.65" rpy="0 0 0.0" />
+  </xacro:sensor_d435>
+  <!-- <xacro:sensor_d435 name="camera_right" topics_ns="camera_right" parent="front_center" publish_pointcloud="true">
+    <origin xyz="0.5 -0.13 0.0" rpy="0 0 -0.15" />
+  </xacro:sensor_d435>   -->
 </robot>
